File: LittleBox_3.kicad_pcb (KiCad board)
At the start: 2 copper layers, 52 parts, among them P1 CONN_2, P2 CONN_2, P3 CONN_15, P4 CONN_15, P5 CONN_2, P6 CONN_2, Q1 SPW47N60C3, Q2 SPW47N60C3, Q3 SPW47N60C3, Q4 SPW47N60C3, Q5 IPA65R660CFD, Q6 IPA65R660CFD, Q7 IPA65R660CFD, Q8 IPA65R660CFD, U1 IR25750, U2 IR25750

Commit message: Layout stabilisé
Parts:
- removed F1, F2: FUSE, FUSE6-31
- added C10: 4.7u, Capacitors_SMD:C_0603, F.Cu at (99.8, 66.4)
- added C11: 4.7u, Capacitors_SMD:C_0603, F.Cu at (147.8, 100.7)
- added C12: 100n, Capacitors_SMD:C_0603, F.Cu at (200.4, 60.6)
- added C13: 4.7u, Capacitors_SMD:C_0603, F.Cu at (109.0, 67.1)
- added C14: 4.7u, Capacitors_SMD:C_0603, F.Cu at (115.8, 55.2)
- added C15: 100n, Capacitors_SMD:C_0603, F.Cu at (103.1, 54.4)
- added C16: 1u, Capacitors_SMD:C_0603, F.Cu at (144.7, 132.7)
- added C17: 100n, Capacitors_SMD:C_0603, F.Cu at (150.5, 132.1)
- added C18: 4.7u, Capacitors_SMD:C_0603, F.Cu at (187.1, 44.3)
- added C20: 100n, Capacitors_SMD:C_0603, F.Cu at (234.4, 101.7)
- added C21: 4.7u, Capacitors_SMD:C_0603, F.Cu at (204.5, 92.1)
- added C22: 4.7u, Capacitors_SMD:C_0603, F.Cu at (204.5, 85.6)
- added C23: 1n 1000V, inverter:C_Rect_L12_W5_P6, B.Cu at (183.8, 87.9)
- added C24: 2.2uF 630V, inverter:C_Rect_W15_L32_P27.5, B.Cu at (203.5, 59.0)
- added C25: 1n 1000V, inverter:C_Rect_L12_W5_P6, B.Cu at (184.3, 61.8)
- added C26: 4.7u, Capacitors_SMD:C_0603, F.Cu at (189.7, 56.1)
- added C27: 4.7u, Capacitors_SMD:C_0603, F.Cu at (189.9, 62.9)
- added C28: 1u, Capacitors_SMD:C_0603, F.Cu at (193.5, 129.6)
- added C29: 4.7u, Capacitors_SMD:C_0603, F.Cu at (219.4, 55.5)
- added C30: 4.7u, Capacitors_SMD:C_0603, F.Cu at (232.2, 89.0)
- added C31: 4.7u, Capacitors_SMD:C_0603, F.Cu at (239.8, 89.0)
- added C32: 4.7u, Capacitors_SMD:C_0603, F.Cu at (236.3, 61.1)
- added C33: 4.7u, Capacitors_SMD:C_0603, F.Cu at (243.1, 61.1)
- added C34: 100n, Capacitors_SMD:C_0603, F.Cu at (254.0, 70.2)
- added C36: 100n, Capacitors_SMD:C_0603, F.Cu at (254.0, 74.5)
- added C37: 100n, Capacitors_SMD:C_0603, F.Cu at (254.0, 72.2)
- added C38: 100n, Capacitors_SMD:C_0603, F.Cu at (216.7, 56.2)
- added C39: 100n, Capacitors_SMD:C_0603, F.Cu at (217.9, 52.4)
- added C40: 1u, Capacitors_SMD:C_0603, F.Cu at (182.6, 121.4)
- added C41: 1u, Capacitors_SMD:C_0603, F.Cu at (113.2, 124.2)
- added C42: 1u, Capacitors_SMD:C_0603, F.Cu at (201.0, 121.3)
- added C43: 100n, Capacitors_SMD:C_0603, F.Cu at (77.5, 46.3)
- added C44: 100n, Capacitors_SMD:C_0603, F.Cu at (77.5, 50.1)
- added C45: 100n, Capacitors_SMD:C_0603, F.Cu at (236.5, 49.5)
- added C46: 2.2uF 630V, inverter:C_Rect_W15_L32_P27.5, B.Cu at (77.5, 91.0)
- added C47: 0.1u, Capacitors_SMD:C_0603, F.Cu at (157.0, 54.8)
- added C48: 2.2uF 630V, inverter:C_Rect_W15_L32_P27.5, B.Cu at (78.5, 63.1)
- added C4M1: 100n, Capacitors_SMD:C_0603, F.Cu at (149.4, 114.2)
- added C5M1: 10n, Capacitors_SMD:C_0603, F.Cu at (128.4, 121.0)
- added C6M1: 1u, Capacitors_SMD:C_0603, F.Cu at (130.8, 121.0)
- added C9: 0.1u, Capacitors_SMD:C_0603, F.Cu at (156.6, 51.9)
- added D2: C3D06060A, Diodes_ThroughHole:Diode_TO-220_Vertical, B.Cu at (117.9, 75.0)
- added D4: C3D06060A, Diodes_ThroughHole:Diode_TO-220_Vertical, B.Cu at (166.1, 69.7)
- added L7: 1.2m, inverter:TOROID_15_44_22, B.Cu at (203.5, 98.1)
- added L8: 2u, inverter:BEAD-5, F.Cu at (124.8, 123.1)
- added L9: 330uH, inverter:2100HT-471-V-RC, B.Cu at (77.5, 76.8)
- added P10: CONN_01X03, Pin_Headers:Pin_Header_Straight_1x03, F.Cu at (149.5, 54.1)
- added P11: CONN_01X01, Connect:PINTST, F.Cu at (229.9, 102.8)
- added P12: CONN_01X01, Connect:PINTST, F.Cu at (226.1, 102.4)
- added P12IN1: CONN_1, inverter:FASTON_110-1, F.Cu at (111.8, 139.0)
- added P12_GND1: CONN_1, inverter:FASTON_110-1, F.Cu at (101.1, 138.8)
- added P13: CONN_01X03, Pin_Headers:Pin_Header_Straight_1x03, F.Cu at (222.5, 48.8)
- added P14: CONN_01X01, Connect:PINTST, F.Cu at (246.4, 55.4)
- added P15: CONN_01X01, Connect:PINTST, F.Cu at (246.4, 52.4)
- added P16: CONN_01X03, Pin_Headers:Pin_Header_Straight_1x03, F.Cu at (91.7, 51.6)
- added P17: CONN_01X03, Pin_Headers:Pin_Header_Straight_1x03, F.Cu at (258.8, 77.8)
- added P18: CONN_01X01, Pin_Headers:Pin_Header_Straight_1x01, F.Cu at (243.0, 106.7)
- added P19: CONN_01X03, Pin_Headers:Pin_Header_Straight_1x03, F.Cu at (258.8, 67.1)
- added P20: CONN_01X01, Socket_Strips:Socket_Strip_Straight_1x01, F.Cu at (248.2, 60.0)
- added P21: CONN_01X01, Pin_Headers:Pin_Header_Straight_1x01, F.Cu at (116.8, 69.9)
- added P400IN+1: CONN_1, inverter:FASTON250_Slanted30-1, B.Cu at (69.8, 49.4)
- added P400IN-1: CONN_1, inverter:FASTON250_Slanted30-1, B.Cu at (69.3, 105.7)
- added P5IN1: CONN_1, inverter:FASTON_110-1, F.Cu at (199.1, 139.3)
- added P5_GND1: CONN_1, inverter:FASTON_110-1, F.Cu at (191.8, 139.3)
- added P7: CONN_01X01, Connect:PINTST, F.Cu at (197.9, 66.8)
- added P8: CONN_01X01, Connect:PINTST, F.Cu at (196.4, 81.4)
- added P9: CONN_01X03, Pin_Headers:Pin_Header_Straight_1x03, F.Cu at (148.1, 93.9)
- added POUT1: CONN_1, inverter:FASTON250_Slanted30-1, F.Cu at (252.7, 48.8)
- added POUT2: CONN_1, inverter:FASTON250_Slanted30-1, F.Cu at (251.7, 90.0)
- added P_led1: CONN_2, Pin_Headers:Pin_Header_Straight_1x02, F.Cu at (167.5, 135.8)
- added Pi2c_1: CONN_4, Pin_Headers:Pin_Header_Straight_1x04, F.Cu at (159.0, 131.1)
- added Pi2c_2: CONN_4, Pin_Headers:Pin_Header_Straight_1x04, F.Cu at (163.2, 131.2)
- added Pprog1: CONN_6, Pin_Headers:Pin_Header_Straight_1x06, F.Cu at (100.8, 132.6)
- added Psense1: CONN_1, inverter:FASTON_110-1, F.Cu at (120.2, 139.3)
- added Psense2: CONN_1, inverter:FASTON_110-1, F.Cu at (129.4, 139.0)
- added Pser1: CONN_6, Pin_Headers:Pin_Header_Straight_1x06, F.Cu at (100.9, 128.7)
- added Q10: IPW6045CP, Transistors_TO-247:TO-247_Vertical_Neutral123, B.Cu at (241.3, 78.1)
- added Q9: IPW6045CP, Transistors_TO-247:TO-247_Vertical_Neutral123, B.Cu at (241.3, 69.7)
- added R17: 1, Resistors_SMD:R_0603, F.Cu at (155.0, 85.0)
- added R18: 1k, Resistors_SMD:R_0603, F.Cu at (154.2, 64.9)
- added R19: 1k, Resistors_SMD:R_0603, F.Cu at (154.2, 61.1)
- added R20: 1, Resistors_SMD:R_0603, F.Cu at (149.0, 65.9)
- added R21: 1k, Resistors_SMD:R_0603, F.Cu at (181.7, 83.0)
- added R22: 1, Resistors_SMD:R_0603, F.Cu at (190.1, 82.4)
- added R23: 1k, Resistors_SMD:R_0603, F.Cu at (185.7, 65.6)
- added R24: 1, Resistors_SMD:R_0603, F.Cu at (180.6, 65.6)
- added R25: 1k, Resistors_SMD:R_0603, F.Cu at (223.3, 82.1)
- added R26: 1, Resistors_SMD:R_0603, F.Cu at (226.3, 82.1)
- added R27: 1, Resistors_SMD:R_0603, F.Cu at (223.5, 62.8)
- added R28: 1k, Resistors_SMD:R_0603, F.Cu at (223.5, 65.4)
- added R29: 1, Resistors_SMD:R_0603, F.Cu at (243.6, 81.9)
- added R30: 1k, Resistors_SMD:R_0603, F.Cu at (240.5, 81.9)
- added R31: 22K, Resistors_SMD:R_0603, F.Cu at (137.9, 132.4)
- added R32: 4.7M, Resistors_SMD:R_0603, F.Cu at (251.5, 55.4)
- added R33: 1, Resistors_SMD:R_0603, F.Cu at (237.5, 65.6)
- added R34: 1k, Resistors_SMD:R_0603, F.Cu at (240.8, 65.6)
- added R35: 4.7M, Resistors_SMD:R_0603, F.Cu at (243.6, 101.4)
- added R36: 22K, Resistors_SMD:R_0603, F.Cu at (239.8, 101.4)
- added R37: 22K, Resistors_SMD:R_0603, F.Cu at (131.1, 118.0)
- added R38: 4.7M, Resistors_SMD:R_0603, F.Cu at (116.6, 65.9)
- added SW1: SW_PUSH, Buttons_Switches_SMD:SW_SPST_PTS645, F.Cu at (146.3, 138.2)
- added U10: ADUM3223, Housings_SOIC:SOIC-16_3.9x9.9mm_Pitch1.27mm, F.Cu at (235.7, 94.6)
- added U11: IR25750, Housings_SOT-23_SOT-143_TSOT-6:SOT-23-5, F.Cu at (186.5, 82.6)
- added U13: AZ1117-3.3, SMD_Packages:DPAK-3, F.Cu at (178.4, 128.7)
- added U14: AZ1117-3.3, SMD_Packages:DPAK-3, F.Cu at (112.1, 120.5)
- added U15: 7805, SMD_Packages:DPAK-3, F.Cu at (197.6, 129.9)
- added U16: ADUM3223, Housings_SOIC:SOIC-16_3.9x9.9mm_Pitch1.27mm, F.Cu at (239.6, 55.3)
- added U17: IR25750, Housings_SOT-23_SOT-143_TSOT-6:SOT-23-5, F.Cu at (236.5, 85.9)
- added U18: ACS712, Housings_SOIC:SOIC-8_3.9x4.9mm_Pitch1.27mm, F.Cu at (253.0, 64.8)
- added U19: ACS712, Housings_SOIC:SOIC-8_3.9x4.9mm_Pitch1.27mm, F.Cu at (253.2, 79.8)
- added U20: IR25750, Housings_SOT-23_SOT-143_TSOT-6:SOT-23-5, F.Cu at (219.7, 89.2)
- added U21: ACS712, Housings_SOIC:SOIC-8_3.9x4.9mm_Pitch1.27mm, F.Cu at (83.8, 48.9)
- added U22: STM32F334R8T6, Housings_QFP:LQFP-64_10x10mm_Pitch0.5mm, F.Cu at (140.8, 118.8)
- added U23: ACS712, Housings_SOIC:SOIC-8_3.9x4.9mm_Pitch1.27mm, F.Cu at (218.2, 62.3)
- added U3: DY12D1212-2W, inverter:DY12D1212-2W, F.Cu at (193.9, 49.8)
- added U4: ADUM3223, Housings_SOIC:SOIC-16_3.9x9.9mm_Pitch1.27mm, F.Cu at (198.8, 89.1)
- added U5: ACS712, Housings_SOIC:SOIC-8_3.9x4.9mm_Pitch1.27mm, F.Cu at (153.6, 85.7)
- added U6: ACS712, Housings_SOIC:SOIC-8_3.9x4.9mm_Pitch1.27mm, F.Cu at (155.8, 60.5)
- added U7: B1212LS-1W, inverter:B1212LS-1W, F.Cu at (154.9, 105.6)
- added U8: ADUM3223, Housings_SOIC:SOIC-16_3.9x9.9mm_Pitch1.27mm, F.Cu at (195.2, 59.4)
- added U9: DY12D1212-2W, inverter:DY12D1212-2W, F.Cu at (229.5, 52.7)
- C1, C2, C3: value 2.2uF 600V -> 100n; footprint C-12 -> Capacitors_SMD:C_0603
- C4: value 2.2uF 600V -> 0.1u; footprint C-12 -> Capacitors_SMD:C_0603
- C5: value 1nF -> 0.1u; footprint C2 -> Capacitors_SMD:C_0603
- C6: value 1nF -> 100n; footprint C2 -> Capacitors_SMD:C_0603
- C7, C8: value 1nF -> 0.5u 250V; footprint C2 -> inverter:C_Rect_L18_W8_P15; moved to B.Cu
- D1, D3: footprint TO220_VERT_2 -> Diodes_ThroughHole:Diode_TO-220_Vertical; moved to B.Cu
- D5: value C3D06060A -> LED; footprint TO220_VERT_2 -> LEDs:LED-0603
- D6: value C3D06060A -> SD1206S040S0R5; footprint TO220_VERT_2 -> Diodes_SMD:SOD-323
- L1, L2: value INDUCTOR -> 470uH; footprint L-toroid-8X4 -> inverter:2100HT-471-V-RC; moved to B.Cu
- L3: footprint C2 -> inverter:BEAD-5
- L4: footprint C2 -> inverter:SER20xx-xxxL
- L5: value 1uH -> Bead; footprint C2 -> inverter:BEAD-5
- L6: value Bead -> 1uH; footprint C2 -> inverter:SER20xx-xxxL
- P1, P2, P5, P6: value CONN_2 -> CONN_01X01; footprint bornier2 -> Connect:PINTST
- P3, P4: value CONN_15 -> CONN_01X01; footprint PIN_ARRAY_15X1 -> Socket_Strips:Socket_Strip_Straight_1x01
- Q1, Q2, Q3, Q4: value SPW47N60C3 -> C3M0065090D; footprint TO-247_Vertical_FET-GDS_largePads -> Transistors_TO-247:TO-247_Vertical_Neutral123; moved to B.Cu
- Q5, Q6: value IPA65R660CFD -> C3M0065090D; footprint TO220_VERT_GDS -> Transistors_TO-247:TO-247_Vertical_Neutral123; moved to B.Cu
- Q7, Q8: value IPA65R660CFD -> IPW6045CP; footprint TO220_VERT_GDS -> Transistors_TO-247:TO-247_Vertical_Neutral123; moved to B.Cu
- R1, R3: value 1 -> 0; footprint R4-5 -> Resistors_SMD:R_0603
- R10, R12: value 1k -> 1; footprint R4-5 -> Resistors_SMD:R_0603
- R11, R9: value 1 -> 1k; footprint R4-5 -> Resistors_SMD:R_0603
- R13, R15: value 1 -> 22K; footprint R4-5 -> Resistors_SMD:R_0603
- R14, R16: value 1k -> 4.7M; footprint R4-5 -> Resistors_SMD:R_0603
- R2, R4: value 1k -> 0; footprint R4-5 -> Resistors_SMD:R_0603
- R5, R7: value 1 -> 10k; footprint R4-5 -> Resistors_SMD:R_0603
- R6: value 1k -> 10k; footprint R4-5 -> Resistors_SMD:R_0603
- R8: value 1k -> 510; footprint R4-5 -> Resistors_SMD:R_0603
- U1: value IR25750 -> ADUM3223; footprint SOT23-5 -> Housings_SOIC:SOIC-16_3.9x9.9mm_Pitch1.27mm
- U2: value IR25750 -> B1212LS-1W; footprint SOT23-5 -> inverter:B1212LS-1W
- moved P2 133.3 mm to (110.0, 57.5), turned to 0 degrees
- moved U1 129.7 mm to (102.9, 60.5)
- moved C7 114.7 mm to (122.9, 49.6), turned to 180 degrees
- moved L1 110.9 mm to (137.9, 76.8)
- moved D1 110.7 mm to (105.2, 83.4)
- moved L2 109.7 mm to (137.9, 55.4)
- moved P6 105.5 mm to (199.0, 81.3), turned to 0 degrees
- moved U2 104.1 mm to (122.4, 59.0), turned to 0 degrees
- moved Q2 103.0 mm to (104.1, 75.0), turned to 0 degrees
- moved Q1 102.2 mm to (117.9, 83.4), turned to 180 degrees
- moved Q7 94.8 mm to (223.5, 69.7), turned to 0 degrees
- moved L4 93.8 mm to (168.7, 53.7), turned to 0 degrees
- moved P5 92.6 mm to (194.7, 66.7), turned to 0 degrees
- moved R12 89.5 mm to (103.4, 67.6), turned to 270 degrees
- moved Q8 89.3 mm to (223.5, 78.1), turned to 180 degrees
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Connections:
- C1 pad 1: VCC400 -> /inverter_microcontroller/VSS
- C1 pad 2: GND -> /inverter_microcontroller/VDD
- C2 pad 1: N-0000026 -> /inverter_microcontroller/VSS
- C2 pad 2: GND -> /inverter_microcontroller/VDD
- C3 pad 1: N-0000035 -> /inverter_microcontroller/VSS
- C3 pad 2: GND -> /inverter_microcontroller/VDD
- C4 pad 1: VCC200 -> VCC3_A
- C4 pad 2: GND -> GND_A
- C5 pad 1: /B1 -> Net-(C5-Pad1)
- C5 pad 2: GND -> GND_A
- C6 pad 1: VCC400 -> VDD3_D
- C6 pad 2: /B1 -> GND_P
- C7 pad 1: /B2 -> Net-(C7-Pad1)
- C7 pad 2: GND -> GND_P
- C8 pad 1: VCC400 -> Net-(C8-Pad1)
- C8 pad 2: /B2 -> GND_P
- D1 pad 1: /SSO1H -> Net-(D1-Pad1)
- D1 pad 2: N-0000031 -> V400+
- D3 pad 1: N-0000031 -> Net-(D3-Pad1)
- D3 pad 2: N-0000030 -> Net-(C21-Pad1)
- D5 pad 1: /SSO2H -> Net-(D5-Pad1)
- D5 pad 2: N-0000032 -> GND_P
- D6 pad 1: N-0000032 -> /inverter_microcontroller/VDD
- D6 pad 2: N-0000044 -> Net-(C5M1-Pad2)
- L1 pad 1: /B1 -> Net-(D1-Pad1)
- L1 pad 2: N-0000035 -> Net-(C7-Pad1)
- L2 pad 1: N-0000026 -> Net-(C8-Pad1)
- L2 pad 2: /B2 -> Net-(C13-Pad1)
- L3 pad 1: N-0000031 -> Net-(D4-Pad2)
- L5 pad 1: /B2 -> Net-(D3-Pad1)
- L5 pad 2: N-0000033 -> Net-(L5-Pad2)
- L6 pad 1: N-0000033 -> /B1
- L6 pad 2: N-0000032 -> Net-(L5-Pad2)
- P1 pad 1: GND -> /ON225
- P2 pad 1: N-0000024 -> /PB12
- P3 pad 1: GND -> /PA1
- P4 pad 1: /GSW2L -> /PA6
- P5 pad 1: /B1 -> /PA11
- P6 pad 1: N-0000026 -> /PA10
- Q1 pad 1: /B1 -> Net-(Q1-Pad1)
- Q1 pad 2: N-0000027 -> Net-(D1-Pad1)
- Q1 pad 3: GND -> GND_P
- Q2 pad 1: VCC400 -> Net-(Q2-Pad1)
- Q2 pad 2: N-0000040 -> V400+
- Q2 pad 3: /B1 -> Net-(C13-Pad1)
- Q3 pad 1: /B2 -> Net-(Q3-Pad1)
- Q3 pad 2: N-0000037 -> V225
- Q3 pad 3: GND -> Net-(C21-Pad1)
- Q4 pad 1: VCC400 -> Net-(Q4-Pad1)
- Q4 pad 2: N-0000043 -> Net-(D4-Pad1)
- Q4 pad 3: /B2 -> V175
- R1 pad 1: /GSW1L -> /PB15
- R1 pad 2: N-0000027 -> /M_I225
- R10 pad 1: N-000005 -> Net-(R10-Pad1)
- R10 pad 2: VCC200 -> Net-(Q1-Pad1)
- R11 pad 1: N-000004 -> Net-(Q2-Pad1)
- R11 pad 2: /GSO1H -> Net-(C13-Pad1)
- R12 pad 1: /SSO1H -> Net-(R12-Pad1)
- R12 pad 2: N-000004 -> Net-(Q2-Pad1)
- R13 pad 1: /GSO2L -> GND_A
- R13 pad 2: N-0000041 -> /PA1
- R14 pad 1: VCC200 -> /PA1
- R14 pad 2: N-0000041 -> Net-(C8-Pad1)
- R15 pad 1: N-0000042 -> GND_A
- R15 pad 2: /GSO2H -> /PA6
- R16 pad 1: N-0000042 -> /PA6
- R16 pad 2: /SSO2H -> Net-(C7-Pad1)
- R2 pad 1: (no net) -> /PB15
- R2 pad 2: (no net) -> /M_IOUT1
- R3 pad 1: /GSW1H -> /PB14
- R3 pad 2: N-0000040 -> /M_I175
- R4 pad 1: /B1 -> /PB14
- R4 pad 2: N-0000040 -> /M_IOUT2
- R5 pad 1: N-0000037 -> /inverter_microcontroller/PD2
- R5 pad 2: /GSW2L -> Net-(Psense1-Pad1)
- R6 pad 1: GND -> Net-(Psense2-Pad1)
- R6 pad 2: N-0000037 -> GND_P
- R7 pad 1: N-0000043 -> /inverter_microcontroller/BOO0
- R7 pad 2: /GSW2H -> GND_P
- R8 pad 1: /B2 -> /PA5
- R8 pad 2: N-0000043 -> Net-(D5-Pad1)
- R9 pad 1: /GSO1L -> Net-(Q1-Pad1)
- R9 pad 2: N-000005 -> GND_P
- U1 pad 1: /CS1L -> /PB12
- U1 pad 2: (no net) -> /ON225
- U1 pad 3: N-0000027 -> VDD3_D
- U1 pad 4: GND -> GND_P
- U1 pad 5: /B1 -> DIS
- U2 pad 1: /CS2L -> VCC12
- U2 pad 2: (no net) -> GND_12
- U2 pad 4: GND -> Net-(C13-Pad2)
Routing:
- net GND: track 397.9 -> 0.00 mm
- net VCC200: track 219.4 -> 0.00 mm
- net /B2: track 182.5 -> 0.00 mm, vias 1 -> 0
- net VCC400: track 174.4 -> 0.00 mm
- net /B1: track 142.5 -> 0.00 mm
- net /SSO2H: track 73.3 -> 0.00 mm
- net /SSO1H: track 66.1 -> 0.00 mm
- net /CS1L: track 48.4 -> 0.00 mm
- net /GSW1L: track 48.2 -> 0.00 mm
- net /CS2L: track 44.9 -> 0.00 mm
- net /GSW2L: track 41.8 -> 0.00 mm
- net /GSO2H: track 34.4 -> 0.00 mm
- net N-0000037: track 30.4 -> 0.00 mm
- net N-0000032: track 30.2 -> 0.00 mm
- net /GSW1H: track 26.5 -> 0.00 mm
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Other:
- copper layers 2 -> 6
- net class 10A added: clearance 0.3, trace_width 3.7, via_dia 3.7, via_drill 2
- net class 12A removed
- net class 3A removed
- net class 5A added: clearance 0.3, trace_width 1.5, via_dia 2.5, via_drill 1.2
- net class 6A removed
- net class Default: clearance 0.254 -> 0.2; trace_width 0.254 -> 0.25; via_dia 0.889 -> 0.6; via_drill 0.635 -> 0.4
- net class PadWidth06 added: clearance 0.2, trace_width 0.6, via_dia 1, via_drill 0.5
- rule pad_to_mask_clearance: 0.2 -> 0
- rule trace_clearance: 0.254 -> 0.2
- rule trace_min: 0.254 -> 0.2
- rule via_min_drill: 0.254 -> 0.3
- rule via_min_size: 0.381 -> 0.4
