File: LittleBox_3_data.kicad_pcb (KiCad board)
At the start: 2 copper layers, 200 x 90 mm, 139 parts, among them P1 CONN_01X01, P10 CONN_01X03, P11 CONN_01X01, P12 CONN_01X01, P12IN1 CONN_1, P12_GND1 CONN_1, P13 CONN_01X03, P14 CONN_01X01, P15 CONN_01X01, P16 CONN_01X03, P17 CONN_01X03, P18 CONN_01X01, P19 CONN_01X03, P2 CONN_01X01, P20 CONN_01X01, P21 CONN_01X01, P22 CONN_01X02, P23 CONN_01X02, P24 CONN_01X02, P25 CONN_01X02, P26 CONN_01X02, P27 CONN_01X02, P28 CONN_01X03, P29 CONN_01X02, P3 CONN_01X01, P30 CONN_01X03, P31 CONN_01X02, P32 CONN_01X03, P4 CONN_01X01, P5 CONN_01X01, P5IN1 CONN_1, P5_GND1 CONN_1, P6 CONN_01X01, P7 CONN_01X01, P8 CONN_01X01, P9 CONN_01X03, Q11 CJ2302, SW1 SW_PUSH, U1 ADUM3223, U10 ADUM3223, U11 IR25750, U12 AZ1117-5, U13 MIC5205-3.3, U14 AZ1117-3.3, U15 MIC5205-5.0, U16 ADUM3223, U17 IR25750, U2 B1212LS-1W, U20 IR25750, U22 STM32F334R8T6, U3 DY12D1212-2W, U4 ADUM3223, U7 B1212LS-1W, U8 ADUM3223, U9 DY12D1212-2W

Commit message: Ajout texte
Other:
- board text added: "Caudos inverter control board V 1 2016 Jose Luu"
Changed lines of the file:
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@@
     (area 37.386904 49.949999 262.613096 140.050001)
     (thickness 1.6)
-    (drawings 31)
+    (drawings 32)
     (tracks 2315)
     (zones 0)
@@
       (solder_mask_margin 0.77) (clearance 0.77))
   )
+  (gr_text "Caudos inverter control board V 1  2016  Jose Luu" (at 111.5 135) (layer F.SilkS)
+    (effects (font (size 1.5 1.5) (thickness 0.3)))
+  )
   (gr_circle (center 150 55) (end 150 56.5) (layer Edge.Cuts) (width 0.1))

Commit message: Indications dans Cmts.User
Other:
- board text added: "<- Hole 3mm diameter"
Changed lines of the file:
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@@
     (area -427.5 -96.5 262.613096 140.050001)
     (thickness 1.6)
-    (drawings 33)
+    (drawings 34)
     (tracks 2315)
     (zones 0)
@@
     (visible_elements 7FFFF77F)
     (pcbplotparams
-      (layerselection 0x010fc_80000001)
+      (layerselection 0x012f8_80000001)
       (usegerberextensions false)
       (excludeedgelayer true)
@@
       (solder_mask_margin 0.77) (clearance 0.77))
   )
+  (gr_text "<- Hole 3mm diameter" (at 92 55) (layer Cmts.User)
+    (effects (font (size 1.5 1.5) (thickness 0.3)))
+  )
   (target plus (at -425 -94) (size 5) (width 0.1) (layer Edge.Cuts))
   (gr_text "Caudos inverter control board V 1  2016  Jose Luu" (at 111.5 135) (layer F.SilkS)
@@
     (effects (font (size 1.5 1.5) (thickness 0.3)))
   )
-  (gr_text "CUT OUT" (at 145.714 72.729) (layer Eco2.User)
+  (gr_text "CUT OUT" (at 145.714 72.729) (layer Cmts.User)
     (effects (font (size 1.5 1.5) (thickness 0.3)))
   )
-  (gr_text "CUT OUT" (at 145.814 112.629) (layer Eco2.User)
+  (gr_text "CUT OUT" (at 145.814 112.629) (layer Cmts.User)
     (effects (font (size 1.5 1.5) (thickness 0.3)))
   )
